File: KiCad/USB-C-Lane1-2.kicad_sch (KiCad schematic)
At the start: 33 parts, among them J1 USB_C_Receptacle

Commit message: WIP - fine tune routing
WIP - fine tune routing
Parts:
- removed C12: 1u, Capacitor_SMD:C_0603_1608Metric_Pad1.08x0.95mm_HandSolder, symbol pcie2usbc-eagle-import:C-EUC0603K
- removed C13: 100n, Capacitor_SMD:C_0603_1608Metric_Pad1.08x0.95mm_HandSolder, symbol pcie2usbc-eagle-import:C-EUC0603K
- removed D2: LED, LED_SMD:LED_0805_2012Metric_Pad1.15x1.40mm_HandSolder, symbol Device:LED
- removed R4: 10k, Resistor_SMD:R_0402_1005Metric_Pad0.72x0.64mm_HandSolder, symbol pcie2usbc-eagle-import:R-US_R0603
- J1: footprint Connector_USB:USB_C_Receptacle_Amphenol_12401548E4-2A -> Connector_USB:USB_C_Receptacle_Amphenol_12401610E4-2A
- renumbered D3 to 3V3_D3, D1 to PERST_D1, R2 to R4, R3 to R5, R5 to R7

Commit message: Layout completed
Layout completed
Parts:
- removed TP5: TPTP38X20, TestPoint:TestPoint_Pad_D1.5mm, symbol pcie2usbc-eagle-import:TPTP38X20
- added TP5: TestPoint, TestPoint:TestPoint_Keystone_5015_Micro-Minature, symbol Connector:TestPoint
Connections:
- net GND: now also TP5.1
Changed lines of the file:
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@@
+    )
+  )
+  (symbol (lib_id "Connector:TestPoint") (at 207.01 62.23 0) (unit 1)
+    (in_bom yes) (on_board yes) (dnp no) (fields_autoplaced)
+    (property "Reference" "TP5" (at 209.55 57.658 0)
+      (effects (font (size 1.27 1.27)) (justify left))
+    )
+    (property "Value" "TestPoint" (at 209.55 60.198 0)
+      (effects (font (size 1.27 1.27)) (justify left))
+    )
+    (property "Footprint" "TestPoint:TestPoint_Keystone_5015_Micro-Minature" (at 212.09 62.23 0)
+      (effects (font (size 1.27 1.27)) hide)
+    )
+    (property "Datasheet" "~" (at 212.09 62.23 0)
+      (effects (font (size 1.27 1.27)) hide)
+    )
+    (pin "1")
+    (instances
+      (project "m-pcie2usbc"
+        (path "/c6966a4c-26ab-49f3-b12b-daf57b153bc7/65aeb514-2985-4b7f-9956-bb6e254cf14f"
+          (reference "TP5") (unit 1)
+        )
+        (path "/c6966a4c-26ab-49f3-b12b-daf57b153bc7/353549ee-224f-4768-b417-4f602901b20c"
+          (reference "TP10") (unit 1)
+        )
+      )
     )
   )
@@
         )
       )
-    )
-  )
-  (symbol (lib_id "pcie2usbc-eagle-import:TPTP38X20") (at 207.01 62.23 0) (unit 1)
-    (in_bom yes) (on_board yes) (dnp no)
-    (property "Reference" "TP5" (at 203.2 62.23 0)
-      (effects (font (size 1.524 1.2954)) (justify right) hide)
-    )
-    (property "Value" "TPTP38X20" (at 207.01 62.23 0)
-      (effects (font (size 1.27 1.27)) hide)
-    )
-    (property "Footprint" "TestPoint:TestPoint_Pad_D1.5mm" (at 207.01 62.23 0)
-      (effects (font (size 1.27 1.27)) hide)
-    )
-    (property "Datasheet" "" (at 207.01 62.23 0)
-      (effects (font (size 1.27 1.27)) hide)
-    )
-    (property "TP_SIGNAL_NAME" "GND" (at 203.2 62.23 0)
-      (effects (font (size 1.27 1.27)) (justify right) hide)
-    )
-    (pin "TP")
-    (instances
-      (project "m-pcie2usbc"
-        (path "/c6966a4c-26ab-49f3-b12b-daf57b153bc7/65aeb514-2985-4b7f-9956-bb6e254cf14f"
-          (reference "TP5") (unit 1)
-        )
-        (path "/c6966a4c-26ab-49f3-b12b-daf57b153bc7/353549ee-224f-4768-b417-4f602901b20c"
-          (reference "TP10") (unit 1)
-        )
-      )
-      (project "pcie2usbc"
-        (path "/e1766754-b9de-4cd8-9e76-5cd3a12f2f48"
-          (reference "TP13") (unit 1)
-        )
-        (path "/e1766754-b9de-4cd8-9e76-5cd3a12f2f48/0780fae0-cf9e-47a3-8386-0708b158015b"
-          (reference "TP14") (unit 1)
-        )
-        (path "/e1766754-b9de-4cd8-9e76-5cd3a12f2f48/265201af-3e4e-4a3b-a1e2-272c609923eb"
-          (reference "TP19") (unit 1)
-        )
-      )
