File: KiCad/m-pcie2usbc.kicad_pcb (KiCad board)
At the start: 2 copper layers, 30 x 51 mm, 72 parts, among them J2 USB_C_Receptacle, J3 USB_C_Receptacle

Commit message: WIP - fine tune routing
WIP - fine tune routing
Parts:
- removed the C14 at (152.1, 105.6)
- removed the C20 at (149.7, 101.2)
- removed C28: 100n, Capacitor_SMD:C_0603_1608Metric_Pad1.08x0.95mm_HandSolder
- removed the C3 at (167.4, 96.9)
- removed D2, D5: LED, LED_SMD:LED_0805_2012Metric_Pad1.15x1.40mm_HandSolder
- removed the D4 at (148.3, 80.8)
- removed the D6 at (148.3, 83.7)
- removed the R4 at (169.2, 78.3)
- removed the R9 at (148.2, 83.7)
- added 3V3_D3: LED, LED_SMD:LED_0805_2012Metric_Pad1.15x1.40mm_HandSolder, F.Cu at (127.4, 77.6)
- added PERST_D1: LED, LED_SMD:LED_0805_2012Metric_Pad1.15x1.40mm_HandSolder, F.Cu at (124.9, 77.6)
- added R2: 10k, Resistor_SMD:R_0201_0603Metric_Pad0.64x0.40mm_HandSolder, B.Cu at (121.4, 91.2)
- added R3: 10k, Resistor_SMD:R_0201_0603Metric_Pad0.64x0.40mm_HandSolder, B.Cu at (113.0, 98.2)
- C1: renamed from C18; footprint Capacitor_SMD:C_0402_1005Metric_Pad0.74x0.62mm_HandSolder -> Capacitor_SMD:C_0603_1608Metric_Pad1.08x0.95mm_HandSolder; moved to B.Cu
- C10: renamed from C17; moved to B.Cu
- C11: renamed from C22; moved to B.Cu
- C14: renamed from C11; value 100n -> 1u; footprint Capacitor_SMD:C_0402_1005Metric_Pad0.74x0.62mm_HandSolder -> Capacitor_SMD:C_0603_1608Metric_Pad1.08x0.95mm_HandSolder; moved to B.Cu
- C15: renamed from C6; footprint Capacitor_SMD:C_0402_1005Metric_Pad0.74x0.62mm_HandSolder -> Capacitor_SMD:C_0603_1608Metric_Pad1.08x0.95mm_HandSolder; moved to B.Cu
- C16: renamed from C27; value 1u -> 100n; moved to B.Cu
- C17: renamed from C10; moved to B.Cu
- C18: renamed from C5; moved to B.Cu
- C19: renamed from C1; footprint Capacitor_SMD:C_0603_1608Metric_Pad1.08x0.95mm_HandSolder -> Capacitor_SMD:C_0402_1005Metric_Pad0.74x0.62mm_HandSolder
- C2: renamed from C12; value 1u -> 100n; footprint Capacitor_SMD:C_0603_1608Metric_Pad1.08x0.95mm_HandSolder -> Capacitor_SMD:C_0402_1005Metric_Pad0.74x0.62mm_HandSolder; moved to B.Cu
- C20: renamed from C16; footprint Capacitor_SMD:C_0603_1608Metric_Pad1.08x0.95mm_HandSolder -> Capacitor_SMD:C_0402_1005Metric_Pad0.74x0.62mm_HandSolder
- C24: renamed from C30; footprint Capacitor_SMD:C_0603_1608Metric_Pad1.08x0.95mm_HandSolder -> Capacitor_SMD:C_0402_1005Metric_Pad0.74x0.62mm_HandSolder
- C26: renamed from C29; value 1u -> 100n; footprint Capacitor_SMD:C_0603_1608Metric_Pad1.08x0.95mm_HandSolder -> Capacitor_SMD:C_0402_1005Metric_Pad0.74x0.62mm_HandSolder
- C29: renamed from C4; value 100n -> 1u; footprint Capacitor_SMD:C_0402_1005Metric_Pad0.74x0.62mm_HandSolder -> Capacitor_SMD:C_0603_1608Metric_Pad1.08x0.95mm_HandSolder; moved to F.Cu
- C3: renamed from C24; moved to B.Cu
- C30: renamed from C15; moved to F.Cu
- C4: renamed from C25; moved to B.Cu
- C5: renamed from C21; moved to B.Cu
- C6: renamed from C23; moved to B.Cu
- C7: renamed from C13; footprint Capacitor_SMD:C_0603_1608Metric_Pad1.08x0.95mm_HandSolder -> Capacitor_SMD:C_0402_1005Metric_Pad0.74x0.62mm_HandSolder; moved to B.Cu
- C8: renamed from C19; moved to B.Cu
- C9: renamed from C26; moved to B.Cu
- J1: renamed from J2; value USB_C_Receptacle -> ~; footprint Connector_USB:USB_C_Receptacle_Amphenol_12401548E4-2A -> M.2-Templates:M.2-M-KEY
- J2: renamed from J3; footprint Connector_USB:USB_C_Receptacle_Amphenol_12401548E4-2A -> Connector_USB:USB_C_Receptacle_Amphenol_12401610E4-2A
- J3: renamed from J1; value ~ -> USB_C_Receptacle; footprint mpcie:mpcie-full-card -> Connector_USB:USB_C_Receptacle_Amphenol_12401610E4-2A
- JP1: renamed from JP14; moved to B.Cu
- JP10: renamed from JP6; moved to B.Cu
- JP2: renamed from JP3; moved to B.Cu
- JP3: renamed from JP4; moved to B.Cu
- JP4: renamed from JP7; moved to B.Cu
- JP5: renamed from JP2; moved to B.Cu
- JP6: renamed from JP8; moved to B.Cu
- JP7: renamed from JP9; moved to B.Cu
- JP8: renamed from JP10; moved to B.Cu
- JP9: renamed from JP5; moved to B.Cu
- R1: renamed from R2; value 100k -> 10k; footprint Resistor_SMD:R_0402_1005Metric_Pad0.72x0.64mm_HandSolder -> Resistor_SMD:R_0201_0603Metric_Pad0.64x0.40mm_HandSolder
- R11: renamed from R1; value 10k -> 2.2k; footprint Resistor_SMD:R_0201_0603Metric_Pad0.64x0.40mm_HandSolder -> Resistor_SMD:R_0402_1005Metric_Pad0.72x0.64mm_HandSolder; moved to F.Cu
- R4: renamed from R3; value 2.2k -> 100k
- R5: renamed from R6; value 100k -> 2.2k; moved to F.Cu
- R7: renamed from R5; moved to F.Cu
- R8: value 10k -> 100k
- R9: renamed from R7; moved to F.Cu
- TP10: renamed from TP5; moved to F.Cu
- TP2: renamed from TP10; value TPTP38X20 -> TestPoint; footprint TestPoint:TestPoint_Pad_D1.5mm -> TestPoint:TestPoint_Pad_1.0x1.0mm
- TP5: renamed from TP3; value TestPoint -> TPTP38X20; footprint TestPoint:TestPoint_Pad_1.0x1.0mm -> TestPoint:TestPoint_Pad_D1.5mm; moved to F.Cu
- TP6: renamed from TP8; moved to F.Cu
- TP7: renamed from TP4; moved to F.Cu
- TP8: renamed from TP2; moved to F.Cu
- TP9: moved to F.Cu
- moved JP8 77.5 mm to (123.3, 52.0), turned to -90 degrees
- moved JP9 77.4 mm to (121.0, 55.8), turned to 180 degrees
- moved JP10 77.4 mm to (123.4, 55.1)
- moved JP7 75.2 mm to (125.1, 51.9)
- moved C16 68.6 mm to (112.0, 70.5), turned to 90 degrees
- moved R11 62.5 mm to (111.9, 94.0), turned to -90 degrees
- moved C24 61.6 mm to (113.4, 91.4), turned to -90 degrees
- moved J3 61.1 mm to (115.6, 79.8)
- moved D6 60.5 mm to (111.8, 97.2), turned to -90 degrees
- moved JP6 59.3 mm to (114.8, 66.1)
- moved C26 59.0 mm to (116.1, 88.9), turned to -90 degrees
- moved D4 57.7 mm to (113.8, 97.2), turned to -90 degrees
- moved C18 57.6 mm to (111.7, 86.6)
- moved C19 57.6 mm to (112.3, 91.4), turned to -90 degrees
- moved TP3 57.1 mm to (126.0, 47.2)
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- renumbered C2 to C21, C9 to C22, C8 to C23, C7 to C25, D3 to D4, D1 to D6, JP13 to JP12, JP1 to JP13, JP12 to JP14, TP6 to TP3, TP7 to TP4
Connections:
- C1 pad 1: /USB-C-Lane1-3/RX1_P -> Net-(J2-SHIELD)
- C1 pad 2: /PER0_P -> GND
- C10 pad 1: /USB-C-Lane1-3/D_P -> /USB-C-Lane1-2/RX2_N
- C10 pad 2: /REFCLK_N -> /PER3_N
- C11 pad 1: /USB-C-Lane1-3/D_N -> /USB-C-Lane1-2/TX2_N
- C11 pad 2: /REFCLK_P -> /PET3_N
- C14 pad 1: /USB-C-Lane1-2/TX2_N -> +3V3
- C14 pad 2: /PET3_N -> GND
- C15 pad 1: /USB-C-Lane1-2/TX2_P -> +3V3
- C15 pad 2: /PET3_P -> GND
- C16 pad 1: +12V -> Net-(J3-SHIELD)
- C17 pad 1: /USB-C-Lane1-2/RX2_N -> /USB-C-Lane1-3/D_P
- C17 pad 2: /PER3_N -> /REFCLK_N
- C18 pad 1: /USB-C-Lane1-2/RX2_P -> /USB-C-Lane1-3/RX1_P
- C18 pad 2: /PER3_P -> /PER0_P
- C19 pad 1: Net-(J2-SHIELD) -> /USB-C-Lane1-3/TX1_P
- C19 pad 2: GND -> /PET0_P
- C2 pad 1: +12V -> /USB-C-Lane1-2/D_P
- C2 pad 2: GND -> /REFCLK_N
- C20 pad 1: Net-(J3-SHIELD) -> /USB-C-Lane1-3/RX2_P
- C20 pad 2: GND -> /PER1_P
- C21 pad 1: /USB-C-Lane1-2/D_P -> /USB-C-Lane1-3/TX2_P
- C21 pad 2: /REFCLK_N -> /PET1_P
- C22 pad 1: /USB-C-Lane1-2/TX1_N -> /USB-C-Lane1-3/D_N
- C22 pad 2: /PET2_N -> /REFCLK_P
- C23 pad 1: /USB-C-Lane1-2/RX1_N -> /USB-C-Lane1-3/RX1_N
- C23 pad 2: /PER2_N -> /PER0_N
- C24 pad 1: +3V3 -> /USB-C-Lane1-3/TX1_N
- C24 pad 2: GND -> /PET0_N
- C25 pad 1: /USB-C-Lane1-2/D_N -> /USB-C-Lane1-3/RX2_N
- C25 pad 2: /REFCLK_P -> /PER1_N
- C26 pad 1: +3V3 -> /USB-C-Lane1-3/TX2_N
- C26 pad 2: GND -> /PET1_N
- C29 pad 1: /USB-C-Lane1-2/TX1_P -> +3V3
- C29 pad 2: /PET2_P -> GND
- C3 pad 1: /USB-C-Lane1-3/TX1_N -> /USB-C-Lane1-2/RX1_P
- C3 pad 2: /PET0_N -> /PER2_P
- C4 pad 1: /USB-C-Lane1-3/RX2_N -> /USB-C-Lane1-2/TX1_P
- C4 pad 2: /PER1_N -> /PET2_P
- C5 pad 1: /USB-C-Lane1-3/TX2_P -> /USB-C-Lane1-2/RX2_P
- C5 pad 2: /PET1_P -> /PER3_P
- C6 pad 1: /USB-C-Lane1-3/RX1_N -> /USB-C-Lane1-2/TX2_P
- C6 pad 2: /PER0_N -> /PET3_P
- C7 pad 1: +12V -> /USB-C-Lane1-2/D_N
- C7 pad 2: GND -> /REFCLK_P
- C8 pad 1: /USB-C-Lane1-3/TX1_P -> /USB-C-Lane1-2/RX1_N
- C8 pad 2: /PET0_P -> /PER2_N
- C9 pad 1: /USB-C-Lane1-3/TX2_N -> /USB-C-Lane1-2/TX1_N
- C9 pad 2: /PET1_N -> /PET2_N
- D4 pad 1: Net-(D3-K) -> Net-(D4-K)
- D6 pad 1: Net-(D1-K) -> Net-(D6-K)
- J2 pad A10: /USB-C-Lane1-3/RX2_P -> /USB-C-Lane1-2/RX2_P
- J2 pad A11: /USB-C-Lane1-3/RX2_N -> /USB-C-Lane1-2/RX2_N
- J2 pad A2: /USB-C-Lane1-3/TX1_P -> /USB-C-Lane1-2/TX1_P
- J2 pad A3: /USB-C-Lane1-3/TX1_N -> /USB-C-Lane1-2/TX1_N
- J2 pad A4: /USB-C-Lane1-3/VBUS -> /USB-C-Lane1-2/VBUS
- J2 pad A5: /USB-C-Lane1-3/CC1 -> /USB-C-Lane1-2/CC1
- J2 pad A6: /USB-C-Lane1-3/D_P -> /USB-C-Lane1-2/D_P
- J2 pad A7: /USB-C-Lane1-3/D_N -> /USB-C-Lane1-2/D_N
- J2 pad A8: /USB-C-Lane1-3/SBU1 -> /USB-C-Lane1-2/SBU1
- J2 pad A9: /USB-C-Lane1-3/VBUS -> /USB-C-Lane1-2/VBUS
- J2 pad B10: /USB-C-Lane1-3/RX1_N -> /USB-C-Lane1-2/RX1_N
- J2 pad B11: /USB-C-Lane1-3/RX1_P -> /USB-C-Lane1-2/RX1_P
- J2 pad B2: /USB-C-Lane1-3/TX2_P -> /USB-C-Lane1-2/TX2_P
- J2 pad B3: /USB-C-Lane1-3/TX2_N -> /USB-C-Lane1-2/TX2_N
- J2 pad B4: /USB-C-Lane1-3/VBUS -> /USB-C-Lane1-2/VBUS
- J2 pad B5: /USB-C-Lane1-3/CC2 -> /USB-C-Lane1-2/CC2
- J2 pad B6: /USB-C-Lane1-3/D_P -> /USB-C-Lane1-2/D_P
- J2 pad B7: /USB-C-Lane1-3/D_N -> /USB-C-Lane1-2/D_N
- J2 pad B8: /USB-C-Lane1-3/SBU2 -> /USB-C-Lane1-2/SBU2
- J2 pad B9: /USB-C-Lane1-3/VBUS -> /USB-C-Lane1-2/VBUS
- J2 pad S1: Net-(J3-SHIELD) -> Net-(J2-SHIELD)
- JP1 pad 1: /VBUS_H -> /PRSNT_SEL
- JP1 pad 2: /USB-C-Lane1-3/VBUS -> /USB-C-Lane1-2/PRSNT2_N
- JP10 pad 1: /PRSNT1 -> /USB-C-Lane1-3/PRSNT2_N
- JP10 pad 2: /USB-C-Lane1-2/SBU2 -> /USB-C-Lane1-3/SBU1
- JP12 pad 1: /USB-C-Lane1-3/CC2 -> /PERST_N
- JP12 pad 2: /PERST_N -> /USB-C-Lane1-3/CC1
- JP13 pad 1: /PRSNT_SEL -> /USB-C-Lane1-3/CC2
- JP13 pad 2: /USB-C-Lane1-2/PRSNT2_N -> /PERST_N
- JP14 pad 1: /PERST_N -> /VBUS_H
- JP14 pad 2: /USB-C-Lane1-3/CC1 -> /USB-C-Lane1-3/VBUS
- JP2 pad 1: /PRSNT_SEL -> /PRSNT1
- JP2 pad 2: /USB-C-Lane1-3/PRSNT2_N -> /PRSNT_SEL
- JP3 pad 1: /PRSNT1 -> /PRSNT_SEL
- JP3 pad 2: /PRSNT_SEL -> /USB-C-Lane1-3/PRSNT2_N
- JP4 pad 1: /PERST_N -> /PRSNT1
- JP4 pad 2: /USB-C-Lane1-2/CC1 -> /PRSNT_SEL
- JP5 pad 1: /PRSNT1 -> /USB-C-Lane1-2/PRSNT2_N
- JP5 pad 2: /PRSNT_SEL -> /USB-C-Lane1-2/SBU1
- JP6 pad 1: /USB-C-Lane1-2/CC2 -> /PRSNT1
- JP6 pad 2: /PERST_N -> /USB-C-Lane1-2/SBU2
- JP7 pad 1: /VBUS_H -> /PERST_N
- JP7 pad 2: /USB-C-Lane1-2/VBUS -> /USB-C-Lane1-2/CC1
- JP8 pad 1: /USB-C-Lane1-3/PRSNT2_N -> /USB-C-Lane1-2/CC2
- JP8 pad 2: /USB-C-Lane1-3/SBU1 -> /PERST_N
- JP9 pad 1: /USB-C-Lane1-2/PRSNT2_N -> /VBUS_H
- JP9 pad 2: /USB-C-Lane1-2/SBU1 -> /USB-C-Lane1-2/VBUS
- R1 pad 1: GND -> Net-(J1-DAS/~{DSS})
- R1 pad 2: Net-(J2-SHIELD) -> +3V3
- R11 pad 1: /CLKREQ_N -> GND
- R11 pad 2: +3V3 -> Net-(D6-K)
- R4 pad 1: /PERST_N -> GND
- R4 pad 2: Net-(D1-K) -> Net-(J2-SHIELD)
- R5 pad 1: GND -> /PERST_N
- R5 pad 2: Net-(J3-SHIELD) -> Net-(PERST_D1-K)
- R7 pad 2: Net-(D3-K) -> Net-(3V3_D3-K)
- R8 pad 2: Net-(D5-K) -> Net-(J3-SHIELD)
- TP2 pad 1: (no net) -> /USB-C-Lane1-2/SBU2
- TP3 pad 1: /USB-C-Lane1-3/SBU1 -> /USB-C-Lane1-2/CC1
- TP4 pad 1: /USB-C-Lane1-3/SBU2 -> /USB-C-Lane1-2/CC2
- TP5 pad 1: /USB-C-Lane1-2/CC1 -> (no net)
- TP6 pad 1: /USB-C-Lane1-3/CC1 -> /USB-C-Lane1-3/SBU1
- TP7 pad 1: /USB-C-Lane1-2/CC2 -> /USB-C-Lane1-3/SBU2
- TP8 pad 1: /USB-C-Lane1-2/SBU2 -> /USB-C-Lane1-3/CC1
Routing:
- net /USB-C-Lane1-3/VBUS: track 0.00 -> 64.3 mm, vias 0 -> 3
- net /PERST_N: track 18.5 -> 70.2 mm, vias 2 -> 4
- net +3V3: track 118.8 -> 68.6 mm, vias 1 -> 3
- net /REFCLK_N: track 0.00 -> 41.3 mm, vias 0 -> 2
- net /REFCLK_P: track 0.00 -> 41.2 mm, vias 0 -> 3
- net /USB-C-Lane1-2/SBU1: track 0.00 -> 25.9 mm, vias 0 -> 3
- net /USB-C-Lane1-3/SBU1: track 3.97 -> 29.9 mm, vias 0 -> 1
- net Net-(J1-DAS/~{DSS}): track 0.00 -> 22.0 mm, vias 0 -> 1
- net /USB-C-Lane1-2/RX2_P: track 0.00 -> 20.9 mm, vias 0 -> 1
- net /USB-C-Lane1-2/RX2_N: track 0.00 -> 20.8 mm, vias 0 -> 1
- net /USB-C-Lane1-3/TX1_N: track 3.29 -> 22.3 mm, vias 0 -> 3
- net /USB-C-Lane1-3/TX1_P: track 3.76 -> 22.3 mm, vias 0 -> 3
- net /USB-C-Lane1-3/D_N: track 5.05 -> 23.5 mm, vias 1 -> 2
- net Net-(J2-SHIELD): track 0.00 -> 15.8 mm
- net /PET0_N: track 28.0 -> 12.9 mm, vias 2 -> 1
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- added copper zone on In1.Cu, net GND
- added copper zone on In2.Cu, net GND
Other:
- board size 30 x 51 mm -> 22 x 60.1 mm
- copper layers 2 -> 4

Commit message: Layout completed
Layout completed
Parts:
- TP10, TP5: value TPTP38X20 -> TestPoint; footprint TestPoint:TestPoint_Pad_D1.5mm -> TestPoint:TestPoint_Keystone_5015_Micro-Minature
- moved TP5 1.06 mm to (117.3, 85.4)
Connections:
- J1 pad 68: (no net) -> unconnected-(J1-NC-Pad68)
- J1 pad MOUNTING-HOLE: (no net) -> GND
- TP10 pad 1: (no net) -> GND
- TP5 pad 1: (no net) -> GND
Routing:
- net Net-(J2-SHIELD): track 15.8 -> 33.5 mm
- net Net-(J3-SHIELD): track 20.4 -> 37.6 mm
- net GND: track 40.6 -> 51.2 mm, vias 8 -> 17
- net (no net): vias 4 -> 3
