File: miniPCIe-KiCad/m-pcie2usbc.kicad_pcb (KiCad board)
At the start: 4 copper layers, 22 x 60.1 mm, 66 parts, among them J2 USB_C_Receptacle, J3 USB_C_Receptacle

Commit message: Layout completed / Readme updar
finalized layout
README.me updated
Routing:
- net /REFCLK_P: vias 3 -> 2
- net (no net): vias 3 -> 0
